Commit message: Back to previous version

File: urdf/macros.xacro (robot description, xacro)
@@ -320,5 +320,5 @@
     <inertial>
       <mass value="1e-5" />
-      <origin xyz="-2.5 1.5 1.75" rpy="0 .57 -0.57"/>
+      <origin xyz="-0.25 0 0.025" rpy="0 0 0"/>
       <inertia ixx="1e-6" ixy="0" ixz="0" iyy="1e-6" iyz="0" izz="1e-6" />
     </inertial>
@@ -327,10 +327,10 @@
     <inertial>
       <mass value="1e-5" />
-      <origin xyz="-2.5 1.5 1.75" rpy="0 .57 -0.57"/>
+      <origin xyz="0 0 0.025" rpy="0 0 0"/>
       <inertia ixx="1e-6" ixy="0" ixz="0" iyy="1e-6" iyz="0" izz="1e-6" />
     </inertial>
   </link>
   <joint name="$(arg robot_name)_left_joint" type="fixed">
-    <origin xyz="-2.5 1.5 1.75" rpy="0 .57 -0.57"/>
+    <origin xyz="0 0 0.035" rpy="0 0 0"/>
     <parent link="$(arg robot_name)_link"/>
     <child link="$(arg robot_name)_camera_link"/>
